File: Documentatie eindpuzzel/Schakeling/Schakeling.kicad_sch (KiCad schematic)
At the start: 33 parts, among them Q1 BC817, Q2 BC817

Commit message: Veel nieuwe aanpassing in de Kicad files ( en ook een paar in de code)
Parts:
- removed UART_Suikertje1: 282841-2, components:TE_282841-2, symbol 282841-2:282841-2
- added R10, R9: (no value), symbol Device:R
- added UART_pins1: (no value), symbol Connector:Conn_01x04_Female
- BOOT1, ENABLE1: value SW_Push -> (none); footprint components:TE_3-1825910-1 -> (none)
- C1, C4: value 0.1u -> (none); footprint Capacitor_SMD:C_0805_2012Metric_Pad1.18x1.45mm_HandSolder -> (none)
- C2: value 220u -> (none); footprint Capacitor_SMD:C_0805_2012Metric_Pad1.18x1.45mm_HandSolder -> (none)
- C3: value 22u -> (none); footprint Capacitor_SMD:C_0805_2012Metric_Pad1.18x1.45mm_HandSolder -> (none)
- Clock_Suikertje1, LCD_Suikertje1: value 282841-4 -> (none); footprint 28241:2828414 -> (none)
- D1, D2: value D -> (none); footprint LED_SMD:LED_0603_1608Metric_Pad1.05x0.95mm_HandSolder -> (none)
- ESP_eindpuzzel1: value ESP-WROOM-32 -> (none); footprint components:MODULE_ESP-WROOM-32 -> (none)
- Keypad_Suikertje1: value 282841-7 -> (none); footprint components:TE_282841-7 -> (none)
- LDO1: value AMS1117 -> (none); footprint components:SOT229P700X180-4N -> (none)
- MicroUSB_Poort1: value USB3090-XX-X_REVE -> (none); footprint components:GCT_USB3090-XX-X_REVE -> (none)
- Q1, Q2: value BC817 -> (none); footprint components:SOT95P230X110-3N -> (none)
- R1, R2, R3, R4, R5, R6: value 1k -> (none); footprint Resistor_SMD:R_0805_2012Metric_Pad1.20x1.40mm_HandSolder -> (none)
- R7, R8: value 10k -> (none); footprint Resistor_SMD:R_0805_2012Metric_Pad1.20x1.40mm_HandSolder -> (none)
- Restart_Button1, Start_Button1: value B3F-4050 -> (none); footprint components:SW_B3F-4050 -> (none)
- STATUS1, STATUS2: value LED -> (none); footprint LED_SMD:LED_0805_2012Metric_Pad1.15x1.40mm_HandSolder -> (none)
- SolenoideRelay1, ZwaailichtRelay1: value SRD-05VDC-SL-C -> (none); footprint components:RELAY_SRD-05VDC-SL-C -> (none)
- Solenoide_Suikertje1, Zwaailicht_Suikertje1: value 282841-2 -> (none); footprint components:TE_282841-2 -> (none)
Connections:
- net 3.3V: now also UART_pins1.1 (Pin_1)
- net GND: now also R10.1, R9.1, UART_pins1.4 (Pin_4)
- net IO13: now also R9.2
- net IO14: now also R10.2
- net at ZwaailichtRelay1.COM: now also Zwaailicht_Suikertje1.2
- net at ZwaailichtRelay1.NC: no longer Zwaailicht_Suikertje1.2
- net TX: now reaches ESP_eindpuzzel1.35 (TXD0)
- net TX: now also UART_pins1.2 (Pin_2)
- net RX: now reaches ESP_eindpuzzel1.34 (RXD0)
- net RX: now also UART_pins1.3 (Pin_3)
- net at Solenoide_Suikertje1.1: now also SolenoideRelay1.NO; no longer SolenoideRelay1.COM
- net at Solenoide_Suikertje1.2: now also SolenoideRelay1.COM; no longer SolenoideRelay1.NC
Other:
- note added: "UART Bridge"
- moved on the sheet: R5, R6, Restart_Button1, Solenoide_Suikertje1, Start_Button1, Zwaailicht_Suikertje1

Commit message: Finale design PCB's
Parts:
- added C5, C6: (no value), symbol Device:C
- renumbered Clock_Suikertje1 to Clock1, D2 to D1, D1 to D2, Keypad_Suikertje1 to Keypad1, LCD_Suikertje1 to LCD1, STATUS2 to LED1, STATUS1 to LED2, ZwaailichtRelay1 to Lamp_Relay1, MicroUSB_Poort1 to MicroUSB1, Q1 to NPN1, Q2 to NPN2, Restart_Button1 to Reset1, SolenoideRelay1 to Slot_Relay1, Solenoide_Suikertje1 to Solenoïde1, Start_Button1 to Start1, Zwaailicht_Suikertje1 to Zwaailicht1
Connections:
- net 5V: now also C6.1
- net GND: now also MicroUSB1.6 (SHIELD), MicroUSB1.7 (SHIELD), MicroUSB1.8 (SHIELD), MicroUSB1.9 (SHIELD), C5.1, C6.2
- net at BOOT1.3, BOOT1.4, ESP_eindpuzzel1.25 (IO0)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: now also C5.2
Other:
- moved on the sheet: BOOT1, LDO1

Commit message: Info schematic geupdate en svg files geplot
Parts:
- BOOT1, ENABLE1: value (none) -> SW_Push; footprint (none) -> components:TE_3-1825910-1
- C1, C4, C5: value (none) -> 0.1u; footprint (none) -> Capacitor_SMD:C_0805_2012Metric_Pad1.18x1.45mm_HandSolder
- C2: value (none) -> 220u; footprint (none) -> Capacitor_SMD:CP_Elec_6.3x7.7
- C3: value (none) -> 22u; footprint (none) -> Capacitor_SMD:C_0805_2012Metric_Pad1.18x1.45mm_HandSolder
- C6: value (none) -> 10u; footprint (none) -> Capacitor_SMD:C_0805_2012Metric_Pad1.18x1.45mm_HandSolder
- Clock1, LCD1: value (none) -> 282841-4; footprint (none) -> 28241:2828414
- D1, D2: value (none) -> D; footprint (none) -> LED_SMD:LED_0603_1608Metric_Pad1.05x0.95mm_HandSolder
- ESP_eindpuzzel1: value (none) -> ESP-WROOM-32; footprint (none) -> components:MODULE_ESP-WROOM-32
- Keypad1: value (none) -> 282841-7; footprint (none) -> components:TE_282841-7
- LDO1: value (none) -> AMS1117; footprint (none) -> components:SOT229P700X180-4N
- LED1, LED2: value (none) -> LED; footprint (none) -> LED_SMD:LED_0805_2012Metric_Pad1.15x1.40mm_HandSolder
- Lamp_Relay1, Slot_Relay1: value (none) -> SRD-05VDC-SL-C; footprint (none) -> components:RELAY_SRD-05VDC-SL-C
- MicroUSB1: value (none) -> USB3090-XX-X_REVE; footprint (none) -> components:GCT_USB3090-XX-X_REVE
- NPN1, NPN2: value (none) -> BC817; footprint (none) -> components:SOT95P230X110-3N
- R1, R10, R2, R3, R4, R5, R6, R9: value (none) -> 1k; footprint (none) -> Resistor_SMD:R_0805_2012Metric_Pad1.20x1.40mm_HandSolder
- R7, R8: value (none) -> 10k; footprint (none) -> Resistor_SMD:R_0805_2012Metric_Pad1.20x1.40mm_HandSolder
- Reset1, Start1: value (none) -> B3F-4050; footprint (none) -> components:SW_B3F-4050
- Solenoïde1, Zwaailicht1: value (none) -> 282841-2; footprint (none) -> components:TE_282841-2
- UART_pins1: value (none) -> Conn_01x04_Female; footprint (none) -> Connector_PinSocket_2.54mm:PinSocket_1x04_P2.54mm_Vertical

Commit message: 3D-view pcb's toegevoegd
Other:
- title: Eindpuzzel schakeling -> Eindpuzzel pcb design
Changed lines of the file:
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@@
   (paper "A4")
   (title_block
-    (title "Eindpuzzel schakeling")
+    (title "Eindpuzzel pcb design")
     (date "2022-05-18")
     (rev "Jona Capelle")
