File: Documentatie UV-slot/Schakeling_UV-Lock/Schakeling_UV-Lock.kicad_sch (KiCad schematic)
At the start: 21 parts, among them Q1 BC817

Commit message: Veel nieuwe aanpassing in de Kicad files ( en ook een paar in de code)
Parts:
- removed UART_Suikertje1: 282841-2, components:TE_282841-2, symbol 282841-2:282841-2
- added UART_pins1: (no value), symbol Connector:Conn_01x04_Female
- BOOT1, ENABLE1: value SW_Push -> (none); footprint components:TE_3-1825910-1 -> (none)
- C1, C4: value 0.1u -> (none); footprint Capacitor_SMD:C_0805_2012Metric_Pad1.18x1.45mm_HandSolder -> (none)
- C2: value 220u -> (none); footprint Capacitor_SMD:C_0805_2012Metric_Pad1.18x1.45mm_HandSolder -> (none)
- C3: value 22u -> (none); footprint Capacitor_SMD:C_0805_2012Metric_Pad1.18x1.45mm_HandSolder -> (none)
- D1: value D -> (none); footprint LED_SMD:LED_0603_1608Metric_Pad1.05x0.95mm_HandSolder -> (none)
- ESP_eindpuzzel1: value ESP-WROOM-32 -> (none); footprint components:MODULE_ESP-WROOM-32 -> (none)
- Keypad_Suikertje1: value 282841-7 -> (none); footprint components:TE_282841-7 -> (none)
- LCD_Suikertje1: value 282841-4 -> (none); footprint 28241:2828414 -> (none)
- LDO1: value AMS1117 -> (none); footprint components:SOT229P700X180-4N -> (none)
- MicroUSB_Poort1: value USB3090-XX-X_REVE -> (none); footprint components:GCT_USB3090-XX-X_REVE -> (none)
- Q1: value BC817 -> (none); footprint components:SOT95P230X110-3N -> (none)
- R1, R2: value 10k -> (none); footprint Resistor_SMD:R_0805_2012Metric_Pad1.20x1.40mm_HandSolder -> (none)
- R3, R4: value 1k -> (none); footprint Resistor_SMD:R_0805_2012Metric_Pad1.20x1.40mm_HandSolder -> (none)
- STATUS1: value LED -> (none); footprint LED_SMD:LED_0805_2012Metric_Pad1.15x1.40mm_HandSolder -> (none)
- UV-Lamp_Relay1: value SRD-05VDC-SL-C -> (none); footprint components:RELAY_SRD-05VDC-SL-C -> (none)
- UV-lamp_Suikertje1: value 282841-2 -> (none); footprint components:TE_282841-2 -> (none)
Connections:
- net 3.3V: now also UART_pins1.1 (Pin_1)
- net GND: now also UART_pins1.4 (Pin_4)
- net RX: now reaches ESP_eindpuzzel1.34 (RXD0)
- net RX: now also UART_pins1.3 (Pin_3)
- net TX: now reaches ESP_eindpuzzel1.35 (TXD0)
- net TX: now also UART_pins1.2 (Pin_2)
- net at UV-lamp_Suikertje1.2: now also UV-Lamp_Relay1.COM; no longer UV-Lamp_Relay1.NC
Other:
- note added: "UART Bridge"
- moved on the sheet: UV-lamp_Suikertje1

Commit message: Finale design PCB's
Parts:
- added C5, C6: (no value), symbol Device:C
- renumbered Keypad_Suikertje1 to Keypad1, LCD_Suikertje1 to LCD1
Connections:
- net 5V: now also C6.1
- net GND: now also MicroUSB_Poort1.6 (SHIELD), MicroUSB_Poort1.7 (SHIELD), MicroUSB_Poort1.8 (SHIELD), MicroUSB_Poort1.9 (SHIELD), C5.1, C6.2
- net at BOOT1.3, BOOT1.4, ESP_eindpuzzel1.25 (IO0)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: now also C5.2
- no-connect marks 24 -> 23
Other:
- moved on the sheet: BOOT1, LDO1

Commit message: Info schematic geupdate en svg files geplot
Parts:
- BOOT1, ENABLE1: value (none) -> SW_Push; footprint (none) -> components:TE_3-1825910-1
- C1, C4, C5: value (none) -> 0.1u; footprint (none) -> Capacitor_SMD:C_0805_2012Metric_Pad1.18x1.45mm_HandSolder
- C2: value (none) -> 220u; footprint (none) -> Capacitor_SMD:CP_Elec_6.3x7.7
- C3: value (none) -> 22u; footprint (none) -> Capacitor_SMD:C_0805_2012Metric_Pad1.18x1.45mm_HandSolder
- C6: value (none) -> 10u; footprint (none) -> Capacitor_SMD:C_0805_2012Metric_Pad1.18x1.45mm_HandSolder
- D1: value (none) -> D; footprint (none) -> LED_SMD:LED_0603_1608Metric_Pad1.05x0.95mm_HandSolder
- ESP_eindpuzzel1: value (none) -> ESP-WROOM-32; footprint (none) -> components:MODULE_ESP-WROOM-32
- Keypad1: value (none) -> 282841-7; footprint (none) -> components:TE_282841-7
- LCD1: value (none) -> 282841-4; footprint (none) -> 28241:2828414
- LDO1: value (none) -> AMS1117; footprint (none) -> components:SOT229P700X180-4N
- MicroUSB_Poort1: value (none) -> USB3090-XX-X_REVE; footprint (none) -> components:GCT_USB3090-XX-X_REVE
- Q1: value (none) -> BC817; footprint (none) -> components:SOT95P230X110-3N
- R1, R2: value (none) -> 10k; footprint (none) -> Resistor_SMD:R_0805_2012Metric_Pad1.20x1.40mm_HandSolder
- R3, R4: value (none) -> 1k; footprint (none) -> Resistor_SMD:R_0805_2012Metric_Pad1.20x1.40mm_HandSolder
- STATUS1: value (none) -> LED; footprint (none) -> LED_SMD:LED_0805_2012Metric_Pad1.15x1.40mm_HandSolder
- UART_pins1: value (none) -> Conn_01x04_Female; footprint (none) -> Connector_PinSocket_2.54mm:PinSocket_1x04_P2.54mm_Vertical
- UV-Lamp_Relay1: value (none) -> SRD-05VDC-SL-C; footprint (none) -> components:RELAY_SRD-05VDC-SL-C
- UV-lamp_Suikertje1: value (none) -> 282841-2; footprint (none) -> components:TE_282841-2
Other:
- company: (none) -> KU Leuven
- title: (none) -> UV-Slot pcb design
- moved on the sheet: LCD1, UART_pins1
